File: hardware/circuit/MiniSeq/MiniSeq.kicad_sch (KiCad schematic)
At the start: 73 parts, among them SW1 SMTS-102, SW10 CLOCK_BTN, SW2 SMTS-102, SW3 SMTS-102, SW4 SMTS-102, SW5 SMTS-102, SW6 SMTS-102, SW7 SMTS-102, SW8 SMTS-102, SW9 RESET_BTN, U1 4017, U2 TL072, U3 TL074

Commit message: v0.1 PCBs
Parts:
- removed SW10: CLOCK_BTN, benjiaomodular:Button_KFC7x7, symbol Switch:SW_DPDT_x2
- removed SW9: RESET_BTN, benjiaomodular:Button_KFC7x7, symbol Switch:SW_DPDT_x2
- added C8: 100nF, Capacitor_SMD:C_0805_2012Metric_Pad1.18x1.45mm_HandSolder, symbol Device:C
- added SW11: RESET_BTN, Button_Switch_Keyboard:SW_Cherry_MX_1.00u_PCB, symbol Switch:SW_Push
- added SW9: CLOCK_BTN, Button_Switch_Keyboard:SW_Cherry_MX_1.00u_PCB, symbol Switch:SW_Push
- C1, C2: footprint Capacitor_SMD:C_0603_1608Metric_Pad1.08x0.95mm_HandSolder -> Capacitor_SMD:C_0805_2012Metric_Pad1.18x1.45mm_HandSolder
Connections:
- net +9V: now also C8.1
- net CV_OUT: now also RV1.2; no longer D11.1 (K)
- net GND: now also C8.2
- net STEP1: now also D11.2 (A); no longer RV1.3
- net STEP2: now also D1.2 (A), R1.2, SW2.2 (B); no longer D13.2 (A), R5.2, SW5.2 (B)
- net STEP3: now also D2.2 (A), R2.2, SW3.2 (B); no longer D1.2 (A), R1.2, SW2.2 (B)
- net STEP4: now also D3.2 (A), R3.2, SW4.2 (B); no longer D14.2 (A), R6.2, SW6.2 (B)
- net STEP5: now also D13.2 (A), R5.2, SW5.2 (B); no longer D2.2 (A), R2.2, SW3.2 (B)
- net STEP6: now also D14.2 (A), R6.2, SW6.2 (B); no longer D15.2 (A), R7.2, SW7.2 (B)
- net STEP7: now also D15.2 (A), R7.2, SW7.2 (B); no longer D3.2 (A), R3.2, SW4.2 (B)
- net at C1.1, D26.2 (A): now also SW11.2
- net at R9.1: now also SW11.1
- net at C2.1, D31.2 (A): now also SW9.2
- net at R12.1: now also SW9.1
- new net: D11.1 (K), RV1.3
- no-connect marks 22 -> 14
Other:
- moved on the sheet: C1, D11, D23, D26, R12, R8, RV1

Commit message: Updated PCBs for v0.1
Parts:
- U1: footprint Package_SO:SOIC-16_3.9x9.9mm_P1.27mm -> Package_SO:SOIC-16W_5.3x10.2mm_P1.27mm
Changed lines of the file:
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@@
 			)
 		)
-		(property "Footprint" "Package_SO:SOIC-16_3.9x9.9mm_P1.27mm"
+		(property "Footprint" "Package_SO:SOIC-16W_5.3x10.2mm_P1.27mm"
 			(at 147.32 152.4 0)
 			(effects
